Commit message: feat(description): pass inversion parameters to ros2_control

File: ros2_ws/src/mobile_robot_description/urdf/mobile_robot.ros2_control.xacro (robot description, xacro)
@@ -1,5 +1,5 @@
 <?xml version="1.0"?>
 <robot xmlns:xacro="http://www.ros.org/wiki/xacro">
-  <xacro:macro name="mobile_robot_ros2_control" params="name serial_device baud_rate ticks_per_revolution">
+  <xacro:macro name="mobile_robot_ros2_control" params="name serial_device baud_rate ticks_per_revolution left_motor_inverted right_motor_inverted left_encoder_inverted right_encoder_inverted">
     <ros2_control name="${name}" type="system">
       <hardware>
@@ -7,7 +7,9 @@
         <param name="serial_device">${serial_device}</param>
         <param name="baud_rate">${baud_rate}</param>
-        <param name="io_timeout_ms">20</param>
-        <param name="telemetry_timeout_ms">100</param>
         <param name="ticks_per_revolution">${ticks_per_revolution}</param>
+        <param name="left_motor_inverted">${left_motor_inverted}</param>
+        <param name="right_motor_inverted">${right_motor_inverted}</param>
+        <param name="left_encoder_inverted">${left_encoder_inverted}</param>
+        <param name="right_encoder_inverted">${right_encoder_inverted}</param>
       </hardware>
       <joint name="left_wheel_joint">

Commit message: feat(description): pass telemetry watchdog to hardware

File: ros2_ws/src/mobile_robot_description/urdf/mobile_robot.ros2_control.xacro (robot description, xacro)
@@ -1,5 +1,5 @@
 <?xml version="1.0"?>
 <robot xmlns:xacro="http://www.ros.org/wiki/xacro">
-  <xacro:macro name="mobile_robot_ros2_control" params="name serial_device baud_rate ticks_per_revolution left_motor_inverted right_motor_inverted left_encoder_inverted right_encoder_inverted">
+  <xacro:macro name="mobile_robot_ros2_control" params="name serial_device baud_rate telemetry_timeout_ms ticks_per_revolution left_motor_inverted right_motor_inverted left_encoder_inverted right_encoder_inverted">
     <ros2_control name="${name}" type="system">
       <hardware>
@@ -7,4 +7,5 @@
         <param name="serial_device">${serial_device}</param>
         <param name="baud_rate">${baud_rate}</param>
+        <param name="telemetry_timeout_ms">${telemetry_timeout_ms}</param>
         <param name="ticks_per_revolution">${ticks_per_revolution}</param>
         <param name="left_motor_inverted">${left_motor_inverted}</param>
