Commit message: feat(description): expose telemetry watchdog argument

File: ros2_ws/src/mobile_robot_description/urdf/mobile_robot.urdf.xacro (robot description, xacro)
@@ -3,4 +3,5 @@
   <xacro:arg name="serial_device" default="/dev/serial0"/>
   <xacro:arg name="baud_rate" default="115200"/>
+  <xacro:arg name="telemetry_timeout_ms" default="500"/>
   <xacro:arg name="ticks_per_revolution" default="0.0"/>
   <xacro:arg name="left_motor_inverted" default="false"/>
@@ -28,12 +29,10 @@
   </link>
   <joint name="left_wheel_joint" type="continuous">
-    <parent link="base_link"/>
-    <child link="left_wheel_link"/>
+    <parent link="base_link"/><child link="left_wheel_link"/>
     <origin xyz="0 $(eval float(arg('wheel_separation')) / 2.0) 0" rpy="1.57079632679 0 0"/>
     <axis xyz="0 0 1"/>
   </joint>
   <joint name="right_wheel_joint" type="continuous">
-    <parent link="base_link"/>
-    <child link="right_wheel_link"/>
+    <parent link="base_link"/><child link="right_wheel_link"/>
     <origin xyz="0 $(eval -float(arg('wheel_separation')) / 2.0) 0" rpy="1.57079632679 0 0"/>
     <axis xyz="0 0 1"/>
@@ -43,4 +42,5 @@
     serial_device="$(arg serial_device)"
     baud_rate="$(arg baud_rate)"
+    telemetry_timeout_ms="$(arg telemetry_timeout_ms)"
     ticks_per_revolution="$(arg ticks_per_revolution)"
     left_motor_inverted="$(arg left_motor_inverted)"

Commit message: feat(description): model front and rear caster balls

File: ros2_ws/src/mobile_robot_description/urdf/mobile_robot.urdf.xacro (robot description, xacro)
@@ -1,4 +1,6 @@
 <?xml version="1.0"?>
-<robot xmlns:xacro="http://www.ros.org/wiki/xacro" name="arty_mobile_robot">
+<robot
+  xmlns:xacro="http://www.ros.org/wiki/xacro"
+  name="arty_mobile_robot">
   <xacro:arg name="serial_device" default="/dev/serial0"/>
   <xacro:arg name="baud_rate" default="115200"/>
@@ -9,5 +11,5 @@
   <xacro:arg name="left_encoder_inverted" default="false"/>
   <xacro:arg name="right_encoder_inverted" default="false"/>
-  <xacro:arg name="wheel_radius" default="0.0"/>
+  <xacro:arg name="wheel_radius" default="0.0325"/>
   <xacro:arg name="wheel_separation" default="0.0"/>
   <xacro:arg name="wheel_width" default="0.0"/>
@@ -15,26 +17,116 @@
   <xacro:arg name="base_width" default="0.0"/>
   <xacro:arg name="base_height" default="0.0"/>
-  <xacro:include filename="$(find mobile_robot_description)/urdf/mobile_robot.ros2_control.xacro"/>
+  <xacro:arg name="caster_ball_radius" default="0.0"/>
+  <xacro:arg name="front_caster_offset" default="0.0"/>
+  <xacro:arg name="rear_caster_offset" default="0.0"/>
+  <xacro:include
+    filename="$(find mobile_robot_description)/urdf/mobile_robot.ros2_control.xacro"/>
   <link name="base_link">
-    <visual><geometry><box size="$(arg base_length) $(arg base_width) $(arg base_height)"/></geometry></visual>
-    <collision><geometry><box size="$(arg base_length) $(arg base_width) $(arg base_height)"/></geometry></collision>
+    <visual>
+      <geometry>
+        <box
+          size="$(arg base_length) $(arg base_width) $(arg base_height)"/>
+      </geometry>
+    </visual>
+    <collision>
+      <geometry>
+        <box
+          size="$(arg base_length) $(arg base_width) $(arg base_height)"/>
+      </geometry>
+    </collision>
   </link>
   <link name="left_wheel_link">
-    <visual><geometry><cylinder radius="$(arg wheel_radius)" length="$(arg wheel_width)"/></geometry></visual>
-    <collision><geometry><cylinder radius="$(arg wheel_radius)" length="$(arg wheel_width)"/></geometry></collision>
+    <visual>
+      <geometry>
+        <cylinder
+          radius="$(arg wheel_radius)"
+          length="$(arg wheel_width)"/>
+      </geometry>
+    </visual>
+    <collision>
+      <geometry>
+        <cylinder
+          radius="$(arg wheel_radius)"
+          length="$(arg wheel_width)"/>
+      </geometry>
+    </collision>
   </link>
   <link name="right_wheel_link">
-    <visual><geometry><cylinder radius="$(arg wheel_radius)" length="$(arg wheel_width)"/></geometry></visual>
-    <collision><geometry><cylinder radius="$(arg wheel_radius)" length="$(arg wheel_width)"/></geometry></collision>
+    <visual>
+      <geometry>
+        <cylinder
+          radius="$(arg wheel_radius)"
+          length="$(arg wheel_width)"/>
+      </geometry>
+    </visual>
+    <collision>
+      <geometry>
+        <cylinder
+          radius="$(arg wheel_radius)"
+          length="$(arg wheel_width)"/>
+      </geometry>
+    </collision>
   </link>
-  <joint name="left_wheel_joint" type="continuous">
-    <parent link="base_link"/><child link="left_wheel_link"/>
-    <origin xyz="0 $(eval float(arg('wheel_separation')) / 2.0) 0" rpy="1.57079632679 0 0"/>
+  <link name="front_caster_ball_link">
+    <visual>
+      <geometry>
+        <sphere radius="$(arg caster_ball_radius)"/>
+      </geometry>
+    </visual>
+    <collision>
+      <geometry>
+        <sphere radius="$(arg caster_ball_radius)"/>
+      </geometry>
+    </collision>
+  </link>
+  <link name="rear_caster_ball_link">
+    <visual>
+      <geometry>
+        <sphere radius="$(arg caster_ball_radius)"/>
+      </geometry>
+    </visual>
+    <collision>
+      <geometry>
+        <sphere radius="$(arg caster_ball_radius)"/>
+      </geometry>
+    </collision>
+  </link>
+  <joint
+    name="left_wheel_joint"
+    type="continuous">
+    <parent link="base_link"/>
+    <child link="left_wheel_link"/>
+    <origin
+      xyz="0 $(eval float(arg('wheel_separation')) / 2.0) 0"
+      rpy="1.57079632679 0 0"/>
     <axis xyz="0 0 1"/>
   </joint>
-  <joint name="right_wheel_joint" type="continuous">
-    <parent link="base_link"/><child link="right_wheel_link"/>
-    <origin xyz="0 $(eval -float(arg('wheel_separation')) / 2.0) 0" rpy="1.57079632679 0 0"/>
+  <joint
+    name="right_wheel_joint"
+    type="continuous">
+    <parent link="base_link"/>
+    <child link="right_wheel_link"/>
+    <origin
+      xyz="0 $(eval -float(arg('wheel_separation')) / 2.0) 0"
+      rpy="1.57079632679 0 0"/>
     <axis xyz="0 0 1"/>
+  </joint>
+  <joint
+    name="front_caster_ball_joint"
+    type="fixed">
+    <parent link="base_link"/>
+    <child link="front_caster_ball_link"/>
+    <origin
+      xyz="$(arg front_caster_offset) 0 $(eval -float(arg('wheel_radius')) + float(arg('caster_ball_radius')))"
+      rpy="0 0 0"/>
+  </joint>
+  <joint
+    name="rear_caster_ball_joint"
+    type="fixed">
+    <parent link="base_link"/>
+    <child link="rear_caster_ball_link"/>
+    <origin
+      xyz="$(eval -float(arg('rear_caster_offset'))) 0 $(eval -float(arg('wheel_radius')) + float(arg('caster_ball_radius')))"
+      rpy="0 0 0"/>
   </joint>
   <xacro:mobile_robot_ros2_control
